File: TLPHnodeV2.kicad_pcb (KiCad board)
At the start: 4 copper layers, 28 x 20.5 mm, 35 parts, among them P3 USB (power only), SW1 Reset, U1 NCP703, U2 LD39130S, U3 LPS25HB, U4 Si7006-A20, U5 ESP-12E, U6 ISL29035, U7 bq25070

Commit message: Change board name to TLPHnodeV2
On branch master
modified:   TLPHnodeV2.kicad_pcb
Other:
- board text added: "TLPHnodeV2 2017/01/12"
- board text removed: "TLPHnode 2017/01/12"
Changed lines of the file:
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@@
     (effects (font (size 0.5 0.5) (thickness 0.1)))
   )
-  (gr_text "TLPHnode\n2017/01/12" (at 157.24 83.79 90) (layer F.SilkS)
+  (gr_text "TLPHnodeV2\n2017/01/12" (at 157.24 83.79 90) (layer F.SilkS)
     (effects (font (size 0.5 0.5) (thickness 0.1)))
   )
